File: YE-tangnano9k-EVB.kicad_pcb (KiCad board)
At the start: 2 copper layers, 95 x 72 mm, 23 parts, among them J1 Conn_01x24_Socket, J2 Conn_01x24_Socket, Q1 2SC1815, SW1 SW_SPDT, SW2 SW_Push, SW3 SW_Push, U1 Tang Nano 9K, U2 OSL40391-IRA

Commit message: fix revision date
Other:
- board text added: "rev2025/8/18"
- board text removed: "rev2025/8/6"
Changed lines of the file:
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@@
 		)
 	)
-	(gr_text "rev2025/8/6"
+	(gr_text "rev2025/8/18"
 		(at -39.37 34.29 0)
 		(layer "F.SilkS")
